File: Schematics/Main_Schematic.sch (EAGLE design)
At the start: 35 parts, among them J1 USB_B_PTH

Commit message: Changed names
Other:
- note added: "ATtiny84 Battery V Sens"
Changed lines of the file:
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@@
 <sheet>
 <plain>
-<text x="162.56" y="17.78" size="3.81" layer="94">ATtiny84 HC-SR04 MIM</text>
+<text x="162.56" y="17.78" size="3.81" layer="94">ATtiny84 Battery V Sens</text>
 <text x="182.88" y="10.16" size="3.81" layer="94">1</text>
 <text x="243.84" y="10.16" size="3.81" layer="94">1</text>
